File: Controle-PCB/Controle-PCB.kicad_pcb (KiCad board)
At the start: 2 copper layers, 65 x 45 mm, 7 parts, among them J1 Conn_01x15, J2 Conn_01x02_Male, J3 Conn_01x02_Male, J4 Conn_01x15, J5 Conn_01x03_Male, U1 Teensy3.6_All_Pins

Commit message: PCB changes
Routing:
- net +6V: track 53.3 -> 58.4 mm
- net /3V3: track 11.4 -> 12.7 mm

Commit message: Final version
Parts:
- moved J1 3.05 mm to (121.0, 75.0)
- moved U1 1.00 mm to (140.0, 88.0)
Routing:
- net /3V3: track 12.7 -> 16.5 mm
- net /SCL1: track 8.41 -> 6.36 mm
- net /SDA0: track 7.40 -> 5.35 mm
- net /SCL0: track 7.40 -> 5.35 mm
- net /SDA1: track 8.41 -> 6.36 mm
- net /PWM: track 10.5 -> 9.45 mm
- net /Enable: track 12.0 -> 11.0 mm
- net +6V: track 58.4 -> 57.4 mm
