File: ControlePCB2/ControlePCB2.kicad_pcb (KiCad board)
At the start: 2 copper layers, 65 x 45 mm, 12 parts, among them J1 Conn_01x15_Female, J3 Conn_01x15_Female, U1 GY-521-symbols, U2 GY-521-symbols

Commit message: PCB changes
Routing:
- net +3V3: track 56.3 -> 61.4 mm
- net /SDA1: track 31.8 -> 32.0 mm, vias 1 -> 2
Changed lines of the file:
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@@
     (thickness 1.6)
     (drawings 27)
-    (tracks 20)
+    (tracks 25)
     (zones 0)
     (modules 12)
@@
   )
   (setup
-    (last_trace_width 0.25)
+    (last_trace_width 1)
     (user_trace_width 1)
     (trace_clearance 0.2)
@@
       (effects (font (size 1 1) (thickness 0.15)))
     )
-    (fp_text user %R (at 0.3 0) (layer F.Fab)
-      (effects (font (size 1 1) (thickness 0.15)))
-    )
-    (fp_circle (center 0 0) (end 3.2 0) (layer Cmts.User) (width 0.15))
-    (fp_circle (center 0 0) (end 3.45 0) (layer F.CrtYd) (width 0.05))
+    (fp_circle (center 0 0) (end 3.2 0) (layer Cmts.User) (width 0.15))
+    (fp_circle (center 0 0) (end 3.45 0) (layer F.CrtYd) (width 0.05))
+    (fp_text user %R (at 0.3 0) (layer F.Fab)
+      (effects (font (size 1 1) (thickness 0.15)))
+    )
     (pad 1 np_thru_hole circle (at 0 0) (size 3.2 3.2) (drill 3.2) (layers *.Cu *.Mask))
   )
@@
       (effects (font (size 1 1) (thickness 0.15)))
     )
-    (fp_text user %R (at 0.3 0) (layer F.Fab)
-      (effects (font (size 1 1) (thickness 0.15)))
-    )
-    (fp_circle (center 0 0) (end 3.2 0) (layer Cmts.User) (width 0.15))
-    (fp_circle (center 0 0) (end 3.45 0) (layer F.CrtYd) (width 0.05))
+    (fp_circle (center 0 0) (end 3.2 0) (layer Cmts.User) (width 0.15))
+    (fp_circle (center 0 0) (end 3.45 0) (layer F.CrtYd) (width 0.05))
+    (fp_text user %R (at 0.3 0) (layer F.Fab)
+      (effects (font (size 1 1) (thickness 0.15)))
+    )
     (pad 1 np_thru_hole circle (at 0 0) (size 3.2 3.2) (drill 3.2) (layers *.Cu *.Mask))
   )
@@
       (effects (font (size 1 1) (thickness 0.15)))
     )
-    (fp_text user %R (at 0.3 0) (layer F.Fab)
-      (effects (font (size 1 1) (thickness 0.15)))
-    )
-    (fp_circle (center 0 0) (end 3.2 0) (layer Cmts.User) (width 0.15))
-    (fp_circle (center 0 0) (end 3.45 0) (layer F.CrtYd) (width 0.05))
+    (fp_circle (center 0 0) (end 3.2 0) (layer Cmts.User) (width 0.15))
+    (fp_circle (center 0 0) (end 3.45 0) (layer F.CrtYd) (width 0.05))
+    (fp_text user %R (at 0.3 0) (layer F.Fab)
+      (effects (font (size 1 1) (thickness 0.15)))
+    )
     (pad 1 np_thru_hole circle (at 0 0) (size 3.2 3.2) (drill 3.2) (layers *.Cu *.Mask))
   )
@@
       (effects (font (size 1 1) (thickness 0.15)))
     )
-    (fp_text user %R (at 0.3 0) (layer F.Fab)
-      (effects (font (size 1 1) (thickness 0.15)))
-    )
-    (fp_circle (center 0 0) (end 3.2 0) (layer Cmts.User) (width 0.15))
-    (fp_circle (center 0 0) (end 3.45 0) (layer F.CrtYd) (width 0.05))
+    (fp_circle (center 0 0) (end 3.2 0) (layer Cmts.User) (width 0.15))
+    (fp_circle (center 0 0) (end 3.45 0) (layer F.CrtYd) (width 0.05))
+    (fp_text user %R (at 0.3 0) (layer F.Fab)
+      (effects (font (size 1 1) (thickness 0.15)))
+    )
     (pad 1 np_thru_hole circle (at 0 0) (size 3.2 3.2) (drill 3.2) (layers *.Cu *.Mask))
   )
@@
   (segment (start 146.54 87.2) (end 151.07 91.73) (width 1) (layer F.Cu) (net 2))
   (segment (start 146.54 62) (end 146.54 87.2) (width 1) (layer F.Cu) (net 2))
-  (segment (start 172.38599 93.56401) (end 174.27 91.68) (width 1) (layer F.Cu) (net 2))
-  (segment (start 152.90401 93.56401) (end 172.38599 93.56401) (width 1) (layer F.Cu) (net 2))
-  (segment (start 151.07 91.73) (end 152.90401 93.56401) (width 1) (layer F.Cu) (net 2))
+  (segment (start 151.07 91.73) (end 151.07 94.43) (width 1) (layer F.Cu) (net 2))
+  (segment (start 174.27 91.68) (end 174.27 94.23) (width 1) (layer F.Cu) (net 2))
+  (segment (start 174.27 94.23) (end 172.5 96) (width 1) (layer F.Cu) (net 2))
+  (segment (start 152.64 96) (end 151.07 94.43) (width 1) (layer F.Cu) (net 2))
+  (segment (start 172.5 96) (end 152.64 96) (width 1) (layer F.Cu) (net 2))
   (segment (start 156.049594 91.73) (end 156.15 91.73) (width 1) (layer F.Cu) (net 4))
   (segment (start 151.62 62) (end 151.62 72.12) (width 1) (layer F.Cu) (net 4))
@@
   (segment (start 177 71) (end 182 76) (width 1) (layer B.Cu) (net 14))
   (segment (start 182 91.57) (end 181.89 91.68) (width 1) (layer B.Cu) (net 14))
-  (segment (start 182 76) (end 182 91.57) (width 1) (layer B.Cu) (net 14))
+  (segment (start 182 76) (end 182 76) (width 1) (layer B.Cu) (net 14))
+  (via (at 182 76) (size 1) (drill 0.5) (layers F.Cu B.Cu) (net 14))
+  (segment (start 182 91.57) (end 181.89 91.68) (width 1) (layer F.Cu) (net 14))
+  (segment (start 182 76) (end 182 91.57) (width 1) (layer F.Cu) (net 14))
   (segment (start 179.56 91.47) (end 179.35 91.68) (width 1) (layer F.Cu) (net 15))
   (segment (start 179.56 62) (end 179.56 91.47) (width 1) (layer F.Cu) (net 15))

Commit message: Final version
Parts:
- moved J1 3.00 mm to (144.0, 65.0)
Routing:
- net /SDA1: track 32.0 -> 36.5 mm, vias 2 -> 0
- net /SDA0: track 31.6 -> 28.6 mm
- net /SCL0: track 31.7 -> 28.7 mm
- net +3V3: track 61.4 -> 58.4 mm
- net /SCL1: track 29.8 -> 27.1 mm
