File: Controle-PCB-Arduino/Controle-PCB.kicad_pcb (KiCad board)
At the start: 2 copper layers, 65 x 45 mm, 6 parts, among them J2 Conn_01x02_Male, J3 Conn_01x02_Male, J5 Conn_01x03_Male, U2 GY-521-symbols

Commit message: pcbs
Parts:
- moved J3 2.38 mm to (135.0, 111.0)
Connections:
- A1 pad 13: Net-(A1-Pad13) -> /Enable
- A1 pad 16: /Enable -> Net-(A1-Pad16)
Routing:
- net /Enable: track 7.92 -> 29.5 mm
