File: Controle-PCB-Arduino/Controle-PCB.sch (KiCad schematic (older format))
At the start: 5 parts, among them J2 Conn_01x02_Male, J3 Conn_01x02_Male, J5 Conn_01x03_Male, U2 GY-521-symbols

Commit message: pcbs
Connections:
- net Enable: now also A1.13 (D10); no longer A1.16 (SCK)
Changed lines of the file:
@@
 PWM
 Wire Wire Line
-	5100 4250 4800 4250
-Text Label 4800 4250 0    50   ~ 0
+	5100 3850 4800 3850
+Text Label 4800 3850 0    50   ~ 0
 Enable
 NoConn ~ 5100 2750
@@
 NoConn ~ 5100 3650
 NoConn ~ 5100 3750
-NoConn ~ 5100 3850
 NoConn ~ 5100 4050
 NoConn ~ 5100 4150
@@
 GY-521
 NoConn ~ 6100 3550
+NoConn ~ 5100 4250
 $EndSCHEMATC
