File: Controle-PCB-Arduino-ServoPoweredByNano/Controle-PCB.sch (KiCad schematic (older format))
At the start: 5 parts, among them J2 Conn_01x02_Male, J3 Conn_01x02_Male, J5 Conn_01x03_Male, U2 GY-521-symbols

Commit message: pcbs
Parts:
- removed J2: Conn_01x02_Male, Jupiter:JS-1001-02, symbol Controle-PCB-rescue:Conn_01x02_Male-Connector
Connections:
- net +6V: now also A1.27 (+5V)
- no-connect marks 27 -> 26
Other:
- note removed: "Battery\n"
Changed lines of the file:
@@
 	1    0    0    -1
 $EndComp
-$Comp
-L Controle-PCB-rescue:Conn_01x02_Male-Connector J2
-U 1 1 61E06A34
-P 2350 4350
-AR Path="/61E06A34" Ref="J2"  Part="1"
-AR Path="/61DF7E3D/61E06A34" Ref="J?"  Part="1"
-F 0 "J2" H 2350 4750 50  0000 C CNN
-F 1 "Conn_01x02_Male" H 2350 4650 50  0000 C CNN
-F 2 "Jupiter:JS-1001-02" H 2350 4350 50  0001 C CNN
-F 3 "~" H 2350 4350 50  0001 C CNN
-	1    2350 4350
-	1    0    0    -1
-$EndComp
-$Comp
-L Controle-PCB-rescue:PWR_FLAG-power #FLG0101
-U 1 1 61E06A48
-P 2900 4350
-F 0 "#FLG0101" H 2900 4425 50  0001 C CNN
-F 1 "PWR_FLAG" H 2900 4523 50  0000 C CNN
-F 2 "" H 2900 4350 50  0001 C CNN
-F 3 "~" H 2900 4350 50  0001 C CNN
-	1    2900 4350
-	1    0    0    -1
-$EndComp
-Connection ~ 2900 4350
-Wire Wire Line
-	2550 4350 2900 4350
-$Comp
-L Controle-PCB-rescue:+6V-power #PWR0103
-U 1 1 61E06A56
-P 3150 4350
-F 0 "#PWR0103" H 3150 4200 50  0001 C CNN
-F 1 "+6V" V 3165 4478 50  0000 L CNN
-F 2 "" H 3150 4350 50  0001 C CNN
-F 3 "" H 3150 4350 50  0001 C CNN
-	1    3150 4350
-	0    1    1    0
-$EndComp
-Wire Wire Line
-	2900 4350 3150 4350
 Wire Wire Line
 	2550 3000 3050 3000
@@
 Wire Notes Line
 	1850 3500 1850 2500
-Wire Notes Line
-	1850 3850 3600 3850
 Text Notes 2600 2450 0    50   ~ 0
 Enable\n
-Text Notes 2600 3800 0    50   ~ 0
-Battery\n
 $Comp
 L Connector:Conn_01x03_Male J5
@@
 	1850 1150 3600 1150
 Wire Notes Line
-	3600 2150 3600 1150
+	3650 2350 3650 1350
 Text Notes 2600 1100 0    50   ~ 0
 Servo\n
 Wire Notes Line
-	1850 1150 1850 2150
-Wire Notes Line
-	1850 2150 3600 2150
-$Comp
-L Controle-PCB-rescue:GND-power #PWR0102
-U 1 1 61E06A42
-P 3000 4450
-F 0 "#PWR0102" H 3000 4200 50  0001 C CNN
-F 1 "GND" H 3005 4277 50  0000 C CNN
-F 2 "" H 3000 4450 50  0001 C CNN
-F 3 "" H 3000 4450 50  0001 C CNN
-	1    3000 4450
-	0    -1   -1   0
-$EndComp
-Wire Wire Line
-	2550 4450 3000 4450
-Wire Notes Line
-	3600 4850 3600 3850
-Wire Notes Line
-	1850 4850 3600 4850
-Wire Notes Line
-	1850 4850 1850 3850
+	1900 1350 1900 2350
+Wire Notes Line
+	1900 2350 3650 2350
 Text Label 2300 5600 0    50   ~ 0
 SCL0
@@
 NoConn ~ 6100 3050
 NoConn ~ 6100 2950
-NoConn ~ 5800 2550
 NoConn ~ 5500 2550
 Wire Notes Line
@@
 Wire Notes Line
 	6700 2000 6700 5200
-Wire Notes Line
-	4350 5200 4350 2000
 Text Notes 5350 1950 0    50   ~ 0
 Arduino Nano
-Wire Notes Line
-	6700 5200 4350 5200
 Wire Notes Line
 	1800 5100 3950 5100
@@
 GY-521
 NoConn ~ 6100 3550
+Wire Notes Line
+	6700 5200 4350 5200
+Wire Notes Line
+	4350 5200 4350 2000
+Wire Wire Line
+	5800 2550 5800 2300
+Wire Wire Line
+	5800 2300 6000 2300
+$Comp
+L Controle-PCB-rescue:+6V-power #PWR?
+U 1 1 62519110
+P 6000 2300
+F 0 "#PWR?" H 6000 2150 50  0001 C CNN
+F 1 "+6V" V 6015 2428 50  0000 L CNN
+F 2 "" H 6000 2300 50  0001 C CNN
+F 3 "" H 6000 2300 50  0001 C CNN
+	1    6000 2300
+	0    1    1    0
+$EndComp
 $EndSCHEMATC

Commit message: pcbs
Connections:
- net Enable: now also A1.13 (D10); no longer A1.16 (SCK)
Changed lines of the file:
@@
 Text Label 6400 3850 2    50   ~ 0
 PWM
-Wire Wire Line
-	5100 4250 4800 4250
-Text Label 4800 4250 0    50   ~ 0
-Enable
 NoConn ~ 5100 2750
 NoConn ~ 5100 2850
@@
 NoConn ~ 5100 3650
 NoConn ~ 5100 3750
-NoConn ~ 5100 3850
 NoConn ~ 5100 4050
 NoConn ~ 5100 4150
@@
 	5800 2300 6000 2300
 $Comp
-L Controle-PCB-rescue:+6V-power #PWR?
+L Controle-PCB-rescue:+6V-power #PWR05
 U 1 1 62519110
 P 6000 2300
-F 0 "#PWR?" H 6000 2150 50  0001 C CNN
+F 0 "#PWR05" H 6000 2150 50  0001 C CNN
 F 1 "+6V" V 6015 2428 50  0000 L CNN
 F 2 "" H 6000 2300 50  0001 C CNN
@@
 	0    1    1    0
 $EndComp
+Wire Wire Line
+	5100 3850 4800 3850
+Text Label 4800 3850 0    50   ~ 0
+Enable
+NoConn ~ 5100 4250
 $EndSCHEMATC
