File: Controle-PCB-NyxProject/Projeto Elétrico - Controle.kicad_pcb (KiCad board)
At the start: 2 copper layers, 14 parts, among them J1 Power Supply, J2 Conn_01x03_Male, J3 Conn_01x03_Male, U1 ESP32-DEVKIT-V1, U2 MINI560-StepDown_5v, U3 FlashMemory_W25Q128, U4 GY-521 - Sensor 1, U5 GY-521 - Sensor 2, U6 GY-BMP280

Commit message: -m uploads on PCB and Schematic projects
Connections:
- J2 pad 1: /step_5v+ -> /PWM 1
- J2 pad 2: /PWM 1 -> /step_5v+
- J3 pad 1: /step_5v+ -> /PWM 2
- J3 pad 2: /PWM 2 -> /step_5v+
Routing:
- net /step_5v+: track 108.7 -> 94.4 mm
- net /PWM 1: track 84.3 -> 76.5 mm
- net /PWM 2: track 91.6 -> 85.8 mm
Changed lines of the file:
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@@
     (fp_line (start -2.47 2.55) (end 12.63 2.55) (layer "F.Fab") (width 0.1))
     (pad "1" thru_hole rect (at 0 0 90) (size 3 3) (drill 1.52) (layers *.Cu *.Mask)
-      (net 3 "/step_5v+") (pinfunction "Pin_1") (pintype "passive"))
+      (net 6 "/PWM 2") (pinfunction "Pin_1") (pintype "passive"))
     (pad "2" thru_hole circle (at 5.08 0 90) (size 3 3) (drill 1.52) (layers *.Cu *.Mask)
-      (net 6 "/PWM 2") (pinfunction "Pin_2") (pintype "passive"))
+      (net 3 "/step_5v+") (pinfunction "Pin_2") (pintype "passive"))
     (pad "3" thru_hole circle (at 10.16 0 90) (size 3 3) (drill 1.52) (layers *.Cu *.Mask)
       (net 5 "/step_5v-") (pinfunction "Pin_3") (pintype "passive"))
@@
     (fp_line (start 12.63 -3.75) (end 12.63 3.75) (layer "F.Fab") (width 0.1))
     (pad "1" thru_hole rect (at 0 0 90) (size 3 3) (drill 1.52) (layers *.Cu *.Mask)
-      (net 3 "/step_5v+") (pinfunction "Pin_1") (pintype "passive"))
+      (net 4 "/PWM 1") (pinfunction "Pin_1") (pintype "passive"))
     (pad "2" thru_hole circle (at 5.08 0 90) (size 3 3) (drill 1.52) (layers *.Cu *.Mask)
-      (net 4 "/PWM 1") (pinfunction "Pin_2") (pintype "passive"))
+      (net 3 "/step_5v+") (pinfunction "Pin_2") (pintype "passive"))
     (pad "3" thru_hole circle (at 10.16 0 90) (size 3 3) (drill 1.52) (layers *.Cu *.Mask)
       (net 5 "/step_5v-") (pinfunction "Pin_3") (pintype "passive"))
@@
   (segment (start 92.181 167.132) (end 87.376 162.327) (width 1) (layer "B.Cu") (net 2))
   (segment (start 125.476 167.132) (end 122.936 169.672) (width 1) (layer "B.Cu") (net 2))
-  (segment (start 117.856 144.272) (end 117.944511 144.183489) (width 1) (layer "B.Cu") (net 2))
-  (segment (start 118.381 143.747) (end 117.856 144.272) (width 1) (layer "B.Cu") (net 2))
-  (segment (start 94.996 80.772) (end 92.456 78.232) (width 1) (layer "F.Cu") (net 3))
-  (segment (start 112.776 80.772) (end 94.996 80.772) (width 1) (layer "F.Cu") (net 3))
-  (via (at 112.776 80.772) (size 0.8) (drill 0.4) (layers "F.Cu" "B.Cu") (net 3))
-  (via (at 92.456 78.232) (size 0.8) (drill 0.4) (layers "F.Cu" "B.Cu") (net 3))
-  (segment (start 122.936 101.092) (end 122.936 90.932) (width 1) (layer "B.Cu") (net 3))
-  (segment (start 92.456 73.152) (end 94.996 70.612) (width 1) (layer "B.Cu") (net 3))
-  (segment (start 92.456 78.232) (end 92.456 73.152) (width 1) (layer "B.Cu") (net 3))
-  (segment (start 122.936 90.932) (end 112.776 80.772) (width 1) (layer "B.Cu") (net 3))
-  (segment (start 118.381 105.647) (end 122.936 101.092) (width 1) (layer "B.Cu") (net 3))
-  (segment (start 85.716 70.612) (end 94.996 70.612) (width 1) (layer "B.Cu") (net 3))
-  (segment (start 94.996 70.612) (end 125.476 70.612) (width 1) (layer "B.Cu") (net 3))
-  (segment (start 118.381 113.587) (end 118.381 105.647) (width 1) (layer "B.Cu") (net 3))
-  (segment (start 90.79598 135.459844) (end 90.79598 114.67198) (width 1) (layer "F.Cu") (net 4))
-  (segment (start 92.38801 137.051874) (end 90.79598 135.459844) (width 1) (layer "F.Cu") (net 4))
-  (segment (start 90.79598 114.67198) (end 82.296 106.172) (width 1) (layer "F.Cu") (net 4))
-  (via (at 92.38801 137.051874) (size 0.8) (drill 0.4) (layers "F.Cu" "B.Cu") (net 4))
-  (via (at 82.296 106.172) (size 0.8) (drill 0.4) (layers "F.Cu" "B.Cu") (net 4))
-  (segment (start 87.376 142.007) (end 92.456 136.927) (width 1) (layer "B.Cu") (net 4))
-  (segment (start 82.296 68.952) (end 82.296 106.172) (width 1) (layer "B.Cu") (net 4))
-  (segment (start 85.716 65.532) (end 82.296 68.952) (width 1) (layer "B.Cu") (net 4))
+  (segment (start 117.856 144.272) (end 118.381 143.747) (width 1) (layer "B.Cu") (net 2))
+  (segment (start 128.524 93.472) (end 121.92 86.868) (width 1) (layer "F.Cu") (net 3))
+  (segment (start 121.92 86.868) (end 121.92 76.2) (width 1) (layer "F.Cu") (net 3))
+  (via (at 128.524 93.472) (size 0.8) (drill 0.4) (layers "F.Cu" "B.Cu") (net 3))
+  (via (at 121.92 76.2) (size 0.8) (drill 0.4) (layers "F.Cu" "B.Cu") (net 3))
+  (segment (start 128.524 102.616) (end 128.524 93.472) (width 1) (layer "B.Cu") (net 3))
+  (segment (start 121.412 69.088) (end 121.92 69.088) (width 1) (layer "B.Cu") (net 3))
+  (segment (start 121.92 69.088) (end 125.476 65.532) (width 1) (layer "B.Cu") (net 3))
+  (segment (start 121.92 69.596) (end 121.412 69.088) (width 1) (layer "B.Cu") (net 3))
+  (segment (start 96.012 69.088) (end 121.412 69.088) (width 1) (layer "B.Cu") (net 3))
+  (segment (start 118.381 113.587) (end 118.381 112.759) (width 1) (layer "B.Cu") (net 3))
+  (segment (start 85.716 65.532) (end 92.456 65.532) (width 1) (layer "B.Cu") (net 3))
+  (segment (start 121.92 76.2) (end 121.92 69.596) (width 1) (layer "B.Cu") (net 3))
+  (segment (start 92.456 65.532) (end 96.012 69.088) (width 1) (layer "B.Cu") (net 3))
+  (segment (start 118.381 112.759) (end 128.524 102.616) (width 1) (layer "B.Cu") (net 3))
+  (segment (start 90.424 115.824) (end 90.424 111.76) (width 1) (layer "F.Cu") (net 4))
+  (segment (start 91.44 139.7) (end 90.424 138.684) (width 1) (layer "F.Cu") (net 4))
+  (segment (start 90.424 138.684) (end 90.424 115.824) (width 1) (layer "F.Cu") (net 4))
+  (segment (start 90.424 111.76) (end 85.852 107.188) (width 1) (layer "F.Cu") (net 4))
+  (via (at 85.852 107.188) (size 0.8) (drill 0.4) (layers "F.Cu" "B.Cu") (net 4))
+  (via (at 91.44 139.7) (size 0.8) (drill 0.4) (layers "F.Cu" "B.Cu") (net 4))
+  (segment (start 87.376 142.007) (end 89.133 142.007) (width 1) (layer "B.Cu") (net 4))
+  (segment (start 85.852 70.748) (end 85.716 70.612) (width 1) (layer "B.Cu") (net 4))
+  (segment (start 89.133 142.007) (end 91.44 139.7) (width 1) (layer "B.Cu") (net 4))
+  (segment (start 85.852 107.188) (end 85.852 70.748) (width 1) (layer "B.Cu") (net 4))
   (segment (start 117.856 80.772) (end 117.856 65.532) (width 1) (layer "F.Cu") (net 5))
   (via (at 117.856 80.772) (size 0.8) (drill 0.4) (layers "F.Cu" "B.Cu") (net 5))
@@
   (segment (start 117.856 65.532) (end 117.856 62.992) (width 1) (layer "B.Cu") (net 5))
   (segment (start 117.856 62.992) (end 115.316 60.452) (width 1) (layer "B.Cu") (net 5))
-  (segment (start 110.106479 119.001521) (end 120.396 108.712) (width 1) (layer "F.Cu") (net 6))
-  (segment (start 110.106479 134.241521) (end 110.106479 119.001521) (width 1) (layer "F.Cu") (net 6))
-  (segment (start 130.556 88.392) (end 128.016 90.932) (width 1) (layer "F.Cu") (net 6))
-  (segment (start 107.696 136.652) (end 110.106479 134.241521) (width 1) (layer "F.Cu") (net 6))
-  (segment (start 130.556 78.232) (end 130.556 88.392) (width 1) (layer "F.Cu") (net 6))
-  (via (at 130.556 78.232) (size 0.8) (drill 0.4) (layers "F.Cu" "B.Cu") (net 6))
-  (via (at 107.696 136.652) (size 0.8) (drill 0.4) (layers "F.Cu" "B.Cu") (net 6))
-  (via (at 128.016 90.932) (size 0.8) (drill 0.4) (layers "F.Cu" "B.Cu") (net 6))
-  (via (at 120.396 108.712) (size 0.8) (drill 0.4) (layers "F.Cu" "B.Cu") (net 6))
-  (segment (start 128.016 101.092) (end 120.396 108.712) (width 1) (layer "B.Cu") (net 6))
-  (segment (start 107.696 136.652) (end 107.696 136.927) (width 1) (layer "B.Cu") (net 6))
-  (segment (start 130.556 68.072) (end 130.556 78.232) (width 1) (layer "B.Cu") (net 6))
-  (segment (start 107.696 136.927) (end 112.776 142.007) (width 1) (layer "B.Cu") (net 6))
-  (segment (start 125.476 65.532) (end 128.016 65.532) (width 1) (layer "B.Cu") (net 6))
-  (segment (start 128.016 90.932) (end 128.016 101.092) (width 1) (layer "B.Cu") (net 6))
-  (segment (start 128.016 65.532) (end 130.556 68.072) (width 1) (layer "B.Cu") (net 6))
+  (segment (start 108.712 139.7) (end 109.728 138.684) (width 1) (layer "F.Cu") (net 6))
+  (segment (start 112.776 104.14) (end 113.284 103.632) (width 1) (layer "F.Cu") (net 6))
+  (segment (start 113.284 103.632) (end 121.412 103.632) (width 1) (layer "F.Cu") (net 6))
+  (segment (start 109.728 138.684) (end 109.728 111.252) (width 1) (layer "F.Cu") (net 6))
+  (segment (start 121.412 103.632) (end 122.428 102.616) (width 1) (layer "F.Cu") (net 6))
+  (segment (start 125.476 85.344) (end 125.476 76.708) (width 1) (layer "F.Cu") (net 6))
+  (segment (start 109.728 107.188) (end 112.776 104.14) (width 1) (layer "F.Cu") (net 6))
+  (segment (start 109.728 111.252) (end 109.728 107.188) (width 1) (layer "F.Cu") (net 6))
+  (via (at 125.476 85.344) (size 0.8) (drill 0.4) (layers "F.Cu" "B.Cu") (net 6))
+  (via (at 108.712 139.7) (size 0.8) (drill 0.4) (layers "F.Cu" "B.Cu") (net 6))
+  (via (at 122.428 102.616) (size 0.8) (drill 0.4) (layers "F.Cu" "B.Cu") (net 6))
+  (via (at 125.476 76.708) (size 0.8) (drill 0.4) (layers "F.Cu" "B.Cu") (net 6))
+  (segment (start 112.776 142.007) (end 111.019 142.007) (width 1) (layer "B.Cu") (net 6))
+  (segment (start 122.428 102.616) (end 125.476 99.568) (width 1) (layer "B.Cu") (net 6))
+  (segment (start 111.019 142.007) (end 108.712 139.7) (width 1) (layer "B.Cu") (net 6))
+  (segment (start 125.476 99.568) (end 125.476 85.344) (width 1) (layer "B.Cu") (net 6))
+  (segment (start 125.476 76.708) (end 125.476 70.612) (width 1) (layer "B.Cu") (net 6))
   (segment (start 102.616 98.552) (end 105.156 101.092) (width 1) (layer "F.Cu") (net 7))
   (via (at 102.616 98.552) (size 0.8) (drill 0.4) (layers "F.Cu" "B.Cu") (net 7))

Commit message: Pull-up Resistors added.
Parts:
- added R1: 5K, Resistor_THT:R_Axial_DIN0204_L3.6mm_D1.6mm_P7.62mm_Horizontal, F.Cu at (134.1, 88.5)
- added R2: 5K, Resistor_THT:R_Axial_DIN0204_L3.6mm_D1.6mm_P7.62mm_Horizontal, F.Cu at (130.5, 86.0)
- moved U1 26.3 mm to (121.7, 131.7)
- moved J2 26.3 mm to (107.3, 55.5)
- moved G*** 26.3 mm to (108.4, 75.7)
- moved J1 26.3 mm to (144.5, 149.5)
- moved REF** 26.3 mm to (105.1, 37.7)
- moved REF** 26.3 mm to (105.1, 160.9)
- moved REF** 26.3 mm to (153.4, 37.7)
- moved REF** 26.3 mm to (153.4, 160.9)
- moved U2 26.3 mm to (156.0, 96.5)
- moved U3 26.3 mm to (129.8, 99.6)
- moved U4 26.3 mm to (117.8, 73.7)
- moved U5 26.3 mm to (117.8, 58.5)
- moved U6 26.3 mm to (141.4, 129.4)
- moved J3 26.3 mm to (147.1, 55.5)
Routing:
- net /PWM 2: track 85.8 -> 81.1 mm
- net /3v3: track 146.7 -> 148.8 mm
- net /SDA: track 112.2 -> 111.2 mm
Other:
- board outline added: 56.4 x 131.3 mm

Commit message: First final version
Parts:
- added G***: LOGO, Symbol:Logo_Preto - Copia, F.Cu at (128.8, 73.3)
- added G***: LOGO, Symbol:Logo_Preto - Copia, F.Cu at (214.4, 72.8)
- added J1: Power Supply, TerminalBlock:TerminalBlock_bornier-2_P5.08mm, F.Cu at (166.9, 149.1)
- added J1: Power Supply, TerminalBlock:TerminalBlock_bornier-2_P5.08mm, F.Cu at (252.5, 148.6)
- added J2: Conn_01x03_Male, TerminalBlock:TerminalBlock_bornier-3_P5.08mm, F.Cu at (215.3, 54.6)
- added J2: Conn_01x03_Male, TerminalBlock:TerminalBlock_bornier-3_P5.08mm, F.Cu at (129.7, 55.1)
- added J3: Conn_01x03_Male, TerminalBlock:TerminalBlock_bornier-3_P5.08mm, F.Cu at (255.0, 54.6)
- added J3: Conn_01x03_Male, TerminalBlock:TerminalBlock_bornier-3_P5.08mm, F.Cu at (169.4, 55.1)
- added R1: 5K, Resistor_THT:R_Axial_DIN0204_L3.6mm_D1.6mm_P7.62mm_Horizontal, F.Cu at (156.5, 88.1)
- added R1: 5K, Resistor_THT:R_Axial_DIN0204_L3.6mm_D1.6mm_P7.62mm_Horizontal, F.Cu at (242.1, 87.6)
- added R2: 5K, Resistor_THT:R_Axial_DIN0204_L3.6mm_D1.6mm_P7.62mm_Horizontal, F.Cu at (238.5, 85.1)
- added R2: 5K, Resistor_THT:R_Axial_DIN0204_L3.6mm_D1.6mm_P7.62mm_Horizontal, F.Cu at (152.9, 85.6)
- added REF**: MountingHole_2.2mm_M2, MountingHole:MountingHole_2.2mm_M2, F.Cu at (261.4, 36.8)
- added REF**: MountingHole_2.2mm_M2, MountingHole:MountingHole_2.2mm_M2, F.Cu at (213.1, 160.0)
- added REF**: MountingHole_2.2mm_M2, MountingHole:MountingHole_2.2mm_M2, F.Cu at (127.5, 160.5)
- added REF**: MountingHole_2.2mm_M2, MountingHole:MountingHole_2.2mm_M2, F.Cu at (175.8, 37.3)
- added REF**: MountingHole_2.2mm_M2, MountingHole:MountingHole_2.2mm_M2, F.Cu at (127.5, 37.3)
- added REF**: MountingHole_2.2mm_M2, MountingHole:MountingHole_2.2mm_M2, F.Cu at (261.4, 160.0)
- added REF**: MountingHole_2.2mm_M2, MountingHole:MountingHole_2.2mm_M2, F.Cu at (175.8, 160.5)
- added REF**: MountingHole_2.2mm_M2, MountingHole:MountingHole_2.2mm_M2, F.Cu at (213.1, 36.8)
- added U1: ESP32-DEVKIT-V1, ESP32-DEVKIT-V1:MODULE_ESP32_DEVKIT_V1, F.Cu at (229.6, 130.8)
- added U1: ESP32-DEVKIT-V1, ESP32-DEVKIT-V1:MODULE_ESP32_DEVKIT_V1, F.Cu at (144.0, 131.3)
- added U2: MINI560-StepDown_5v, Jupiter:stepdown 5v, F.Cu at (178.3, 96.1)
- added U2: MINI560-StepDown_5v, Jupiter:stepdown 5v, F.Cu at (263.9, 95.6)
- added U3: FlashMemory_W25Q128, Jupiter:FlashMemory W25Q128, F.Cu at (152.2, 99.2)
- added U3: FlashMemory_W25Q128, Jupiter:FlashMemory W25Q128, F.Cu at (237.8, 98.7)
- added U4: GY-521 - Sensor 1, GY-521:GY-521, F.Cu at (140.2, 73.3)
- added U4: GY-521 - Sensor 1, GY-521:GY-521, F.Cu at (225.8, 72.8)
- added U5: GY-521 - Sensor 2, GY-521:GY-521, F.Cu at (225.8, 57.6)
- added U5: GY-521 - Sensor 2, GY-521:GY-521, F.Cu at (140.2, 58.1)
- added U6: GY-BMP280, Jupiter:GY BMP280, F.Cu at (249.4, 128.5)
- added U6: GY-BMP280, Jupiter:GY BMP280, F.Cu at (163.8, 129.0)
- moved G*** 63.7 mm to (44.7, 72.5)
- moved J1 61.7 mm to (82.8, 148.3)
- moved J2 61.7 mm to (45.6, 54.4)
- moved J3 61.7 mm to (85.3, 54.4)
- moved R2 61.7 mm to (68.8, 84.8)
- moved REF** 61.7 mm to (43.4, 36.6)
- moved REF** 61.7 mm to (43.4, 159.8)
- moved U1 61.7 mm to (59.9, 130.6)
- moved U2 61.7 mm to (94.2, 95.3)
- moved U4 61.7 mm to (56.1, 72.6)
- moved U5 61.7 mm to (56.1, 57.3)
- moved U6 61.7 mm to (79.7, 128.2)
- moved R1 61.7 mm to (72.4, 87.4)
- moved REF** 61.7 mm to (91.7, 36.6)
- moved REF** 61.7 mm to (91.7, 159.8)
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Routing:
- net /3v3: track 148.8 -> 446.3 mm, vias 2 -> 6
- net /SDA: track 111.2 -> 333.6 mm, vias 2 -> 6
- net /SCL: track 106.9 -> 320.6 mm, vias 4 -> 12
- net /step_5v-: track 104.4 -> 313.3 mm, vias 2 -> 6
- net /step_5v+: track 94.4 -> 283.1 mm, vias 2 -> 6
- net VCC: track 83.2 -> 249.7 mm, vias 2 -> 6
- net /PWM 2: track 81.1 -> 243.2 mm, vias 4 -> 12
- net /PWM 1: track 76.5 -> 229.4 mm, vias 2 -> 6
- net /HMOSI: track 61.8 -> 185.5 mm
- net /CS: track 59.6 -> 178.9 mm
- net /HMISO: track 58.0 -> 174.0 mm
- net /HCLK: track 54.1 -> 162.2 mm
- net GND: track 0.51 -> 1.54 mm, vias 1 -> 3
Other:
- board size 56.4 x 131.3 mm -> 226.1 x 132.1 mm

Commit message: PCB files - final version
Parts:
- removed the G*** at (44.7, 72.5)
- removed the G*** at (214.4, 72.8)
- removed the J1 at (252.5, 148.6)
- removed the J1 at (82.8, 148.3)
- removed the J2 at (215.3, 54.6)
- removed the J2 at (45.6, 54.4)
- removed the J3 at (85.3, 54.4)
- removed the J3 at (255.0, 54.6)
- removed the R1 at (242.1, 87.6)
- removed the R1 at (72.4, 87.4)
- removed the R2 at (238.5, 85.1)
- removed the R2 at (68.8, 84.8)
- removed the REF** at (261.4, 36.8)
- removed the REF** at (213.1, 160.0)
- removed the REF** at (91.7, 36.6)
- removed the REF** at (91.7, 159.8)
- removed the REF** at (43.4, 36.6)
- removed the REF** at (261.4, 160.0)
- removed the REF** at (213.1, 36.8)
- removed the REF** at (43.4, 159.8)
- removed the U1 at (59.9, 130.6)
- removed the U1 at (229.6, 130.8)
- removed the U2 at (263.9, 95.6)
- removed the U2 at (94.2, 95.3)
- removed the U3 at (68.1, 98.5)
- removed the U3 at (237.8, 98.7)
- removed the U4 at (225.8, 72.8)
- removed the U4 at (56.1, 72.6)
- removed the U5 at (56.1, 57.3)
- removed the U5 at (225.8, 57.6)
- removed the U6 at (249.4, 128.5)
- removed the U6 at (79.7, 128.2)
- added G***: LOGO, Symbol:Logo_Preto - Copia, F.Cu at (44.9, 69.4)
- added G***: LOGO, Symbol:Logo_Preto - Copia, F.Cu at (212.1, 69.6)
- added J1: Power Supply, TerminalBlock:TerminalBlock_bornier-2_P5.08mm, F.Cu at (250.2, 145.4)
- added J1: Power Supply, TerminalBlock:TerminalBlock_bornier-2_P5.08mm, F.Cu at (83.0, 145.2)
- added J2: Conn_01x03_Male, TerminalBlock:TerminalBlock_bornier-3_P5.08mm, F.Cu at (213.0, 51.4)
- added J2: Conn_01x03_Male, TerminalBlock:TerminalBlock_bornier-3_P5.08mm, F.Cu at (45.7, 51.2)
- added J3: Conn_01x03_Male, TerminalBlock:TerminalBlock_bornier-3_P5.08mm, F.Cu at (252.7, 51.4)
- added J3: Conn_01x03_Male, TerminalBlock:TerminalBlock_bornier-3_P5.08mm, F.Cu at (85.5, 51.2)
- added R1: 5K, Resistor_THT:R_Axial_DIN0204_L3.6mm_D1.6mm_P7.62mm_Horizontal, F.Cu at (72.5, 84.3)
- added R1: 5K, Resistor_THT:R_Axial_DIN0204_L3.6mm_D1.6mm_P7.62mm_Horizontal, F.Cu at (239.8, 84.5)
- added R2: 5K, Resistor_THT:R_Axial_DIN0204_L3.6mm_D1.6mm_P7.62mm_Horizontal, F.Cu at (69.0, 81.7)
- added R2: 5K, Resistor_THT:R_Axial_DIN0204_L3.6mm_D1.6mm_P7.62mm_Horizontal, F.Cu at (236.2, 81.9)
- added REF**: MountingHole_2.2mm_M2, MountingHole:MountingHole_2.2mm_M2, F.Cu at (210.8, 33.7)
- added REF**: MountingHole_2.2mm_M2, MountingHole:MountingHole_2.2mm_M2, F.Cu at (259.1, 156.8)
- added REF**: MountingHole_2.2mm_M2, MountingHole:MountingHole_2.2mm_M2, F.Cu at (43.6, 156.7)
- added REF**: MountingHole_2.2mm_M2, MountingHole:MountingHole_2.2mm_M2, F.Cu at (210.8, 156.8)
- added REF**: MountingHole_2.2mm_M2, MountingHole:MountingHole_2.2mm_M2, F.Cu at (91.8, 156.7)
- added REF**: MountingHole_2.2mm_M2, MountingHole:MountingHole_2.2mm_M2, F.Cu at (91.8, 33.5)
- added REF**: MountingHole_2.2mm_M2, MountingHole:MountingHole_2.2mm_M2, F.Cu at (43.6, 33.5)
- added REF**: MountingHole_2.2mm_M2, MountingHole:MountingHole_2.2mm_M2, F.Cu at (259.1, 33.7)
- added U1: ESP32-DEVKIT-V1, ESP32-DEVKIT-V1:MODULE_ESP32_DEVKIT_V1, F.Cu at (227.3, 127.6)
- added U1: ESP32-DEVKIT-V1, ESP32-DEVKIT-V1:MODULE_ESP32_DEVKIT_V1, F.Cu at (60.1, 127.4)
- added U2: MINI560-StepDown_5v, Jupiter:stepdown 5v, F.Cu at (94.4, 92.2)
- added U2: MINI560-StepDown_5v, Jupiter:stepdown 5v, F.Cu at (261.6, 92.4)
- added U3: FlashMemory_W25Q128, Jupiter:FlashMemory W25Q128, F.Cu at (68.2, 95.4)
- added U3: FlashMemory_W25Q128, Jupiter:FlashMemory W25Q128, F.Cu at (235.5, 95.6)
- added U4: GY-521 - Sensor 1, GY-521:GY-521, F.Cu at (56.3, 69.4)
- added U4: GY-521 - Sensor 1, GY-521:GY-521, F.Cu at (223.5, 69.6)
- added U5: GY-521 - Sensor 2, GY-521:GY-521, F.Cu at (223.5, 54.4)
- added U5: GY-521 - Sensor 2, GY-521:GY-521, F.Cu at (56.3, 54.2)
- added U6: GY-BMP280, Jupiter:GY BMP280, F.Cu at (79.8, 125.1)
- added U6: GY-BMP280, Jupiter:GY BMP280, F.Cu at (247.1, 125.3)
- moved U1 4.34 mm to (142.0, 127.5)
- moved J3 4.34 mm to (167.4, 51.3)
- moved R1 4.34 mm to (154.4, 84.3)
- moved REF** 4.34 mm to (173.7, 33.5)
- moved U2 4.34 mm to (176.3, 92.3)
- moved U3 4.34 mm to (150.1, 95.4)
- moved U4 4.34 mm to (138.2, 69.5)
- moved U5 4.34 mm to (138.2, 54.2)
- moved J1 4.34 mm to (164.8, 145.3)
- moved G*** 4.34 mm to (126.8, 69.4)
- moved REF** 4.34 mm to (125.5, 33.5)
- moved REF** 4.34 mm to (173.7, 156.7)
- moved U6 4.34 mm to (161.7, 125.2)
- moved J2 4.34 mm to (127.6, 51.3)
- moved R2 4.34 mm to (150.9, 81.8)
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Routing:
- net /SDA: track 333.6 -> 341.4 mm
- net /SCL: track 320.6 -> 325.6 mm
- net /step_5v+: track 283.1 -> 286.2 mm
- net /3v3: track 446.3 -> 448.5 mm, vias 6 -> 0
- net /HCLK: track 162.2 -> 163.9 mm
Other:
- board size 226.1 x 132.1 mm -> 223.6 x 131.5 mm
