File: Controle-PCB-GanímedesProject/Projeto Elétrico - ControleGanímedes.kicad_pcb (KiCad board)
At the start: 2 copper layers, 245.9 x 110.4 mm, 39 parts, among them J1 Power Supply, J2 Conn_01x03_Male, J3 Conn_01x03_Male, U1 ESP32-DEVKIT-V1, U3 FlashMemory_W25Q128, U4 GY-521 - Sensor 1, U6 GY-BMP280

Commit message: Update Projeto Elétrico - ControleGanímedes.kicad_pcb
Parts:
- removed the G*** at (39.0, 96.4)
- removed the G*** at (211.7, 96.4)
- removed the J1 at (240.9, 58.8)
- removed the J1 at (68.2, 58.8)
- removed the J1 at (211.1, 129.9)
- removed the J1 at (38.3, 129.9)
- removed the J2 at (215.9, 73.7)
- removed the J2 at (43.2, 73.7)
- removed the J3 at (86.2, 73.7)
- removed the J3 at (258.9, 73.7)
- removed the REF** at (205.9, 153.7)
- removed the REF** at (269.1, 153.7)
- removed the REF** at (33.2, 153.7)
- removed the REF** at (96.4, 53.7)
- removed the REF** at (269.1, 53.7)
- removed the REF** at (205.9, 53.7)
- removed the REF** at (96.4, 153.7)
- removed the REF** at (33.2, 53.7)
- removed the U1 at (246.6, 129.9)
- removed the U1 at (73.9, 129.9)
- removed the U3 at (247.2, 87.7)
- removed the U3 at (74.4, 87.7)
- removed the U4 at (246.6, 96.9)
- removed the U4 at (73.9, 96.9)
- removed the U6 at (269.3, 98.9)
- removed the U6 at (96.5, 98.9)
- added G***: LOGO, Symbol:Logo_Preto - Copia, F.Cu at (211.1, 96.0)
- added G***: LOGO, Symbol:Logo_Preto - Copia, F.Cu at (34.5, 96.0)
- added J1: Power Supply, TerminalBlock:TerminalBlock_bornier-2_P5.08mm, F.Cu at (45.1, 55.9)
- added J1: Power Supply, TerminalBlock:TerminalBlock_bornier-2_P5.08mm, F.Cu at (73.0, 152.4)
- added J1: Power Supply, TerminalBlock:TerminalBlock_bornier-2_P5.08mm, F.Cu at (249.6, 152.4)
- added J1: Power Supply, TerminalBlock:TerminalBlock_bornier-2_P5.08mm, F.Cu at (221.6, 55.9)
- added J2: Conn_01x03_Male, TerminalBlock:TerminalBlock_bornier-3_P5.08mm, F.Cu at (238.1, 152.4)
- added J2: Conn_01x03_Male, TerminalBlock:TerminalBlock_bornier-3_P5.08mm, F.Cu at (61.6, 152.4)
- added J3: Conn_01x03_Male, TerminalBlock:TerminalBlock_bornier-3_P5.08mm, F.Cu at (55.2, 55.9)
- added J3: Conn_01x03_Male, TerminalBlock:TerminalBlock_bornier-3_P5.08mm, F.Cu at (231.8, 55.9)
- added REF**: MountingHole_2.2mm_M2, MountingHole:MountingHole_2.2mm_M2, F.Cu at (28.7, 153.3)
- added REF**: MountingHole_2.2mm_M2, MountingHole:MountingHole_2.2mm_M2, F.Cu at (205.3, 153.3)
- added REF**: MountingHole_2.2mm_M2, MountingHole:MountingHole_2.2mm_M2, F.Cu at (268.5, 53.3)
- added REF**: MountingHole_2.2mm_M2, MountingHole:MountingHole_2.2mm_M2, F.Cu at (91.9, 53.3)
- added REF**: MountingHole_2.2mm_M2, MountingHole:MountingHole_2.2mm_M2, F.Cu at (28.7, 53.3)
- added REF**: MountingHole_2.2mm_M2, MountingHole:MountingHole_2.2mm_M2, F.Cu at (268.5, 153.3)
- added REF**: MountingHole_2.2mm_M2, MountingHole:MountingHole_2.2mm_M2, F.Cu at (205.3, 53.3)
- added REF**: MountingHole_2.2mm_M2, MountingHole:MountingHole_2.2mm_M2, F.Cu at (91.9, 153.3)
- added U1: ESP32-DEVKIT-V1, ESP32-DEVKIT-V1:MODULE_ESP32_DEVKIT_V1, F.Cu at (69.4, 129.5)
- added U1: ESP32-DEVKIT-V1, ESP32-DEVKIT-V1:MODULE_ESP32_DEVKIT_V1, F.Cu at (246.0, 129.5)
- added U3: FlashMemory_W25Q128, Jupiter:FlashMemory W25Q128, F.Cu at (246.5, 87.3)
- added U3: FlashMemory_W25Q128, Jupiter:FlashMemory W25Q128, F.Cu at (70.0, 87.3)
- added U4: GY-521 - Sensor 1, GY-521:GY-521, F.Cu at (69.4, 96.5)
- added U4: GY-521 - Sensor 1, GY-521:GY-521, F.Cu at (246.0, 96.5)
- added U6: GY-BMP280, Jupiter:GY BMP280, F.Cu at (268.6, 98.5)
- added U6: GY-BMP280, Jupiter:GY BMP280, F.Cu at (92.1, 98.5)
- moved J2 82.4 mm to (151.1, 152.4), turned to 180 degrees
- moved J1 45.3 mm to (162.6, 152.4), turned to 0 degrees
- moved J3 31.7 mm to (144.8, 55.9), turned to 0 degrees
- moved J1 18.8 mm to (134.6, 55.9)
Connections:
- U1 pad 4: /HWP -> (no net)
- U1 pad 5: /HHD -> (no net)
- U3 pad 3: /HMOSI -> /HMISO
- U3 pad 6: /HMISO -> /HMOSI
Routing:
- net /PWM 1: track 346.7 -> 34.3 mm, vias 6 -> 0
- net VCC: track 381.2 -> 518.2 mm
- net /HMISO: track 336.3 -> 453.5 mm, vias 6 -> 9
- net /HCLK: track 263.3 -> 341.1 mm
- net /PWM 2: track 507.0 -> 557.5 mm, vias 3 -> 6
- net /CS: track 350.3 -> 359.2 mm
- net /HMOSI: track 402.1 -> 399.1 mm, vias 0 -> 6
- net GND: track 0.00 -> 2.30 mm
Other:
- board size 245.9 x 110.4 mm -> 249.7 x 110 mm

Commit message: PCB Ganimedes embelezada
Parts:
- removed the G*** at (211.1, 96.0)
- removed the G*** at (34.5, 96.0)
- removed the J1 at (45.1, 55.9)
- removed the J1 at (73.0, 152.4)
- removed the J1 at (249.6, 152.4)
- removed the J1 at (221.6, 55.9)
- removed the J2 at (238.1, 152.4)
- removed the J2 at (61.6, 152.4)
- removed the J3 at (55.2, 55.9)
- removed the J3 at (231.8, 55.9)
- removed the REF** at (28.7, 153.3)
- removed the REF** at (205.3, 153.3)
- removed the REF** at (268.5, 53.3)
- removed the REF** at (91.9, 53.3)
- removed the REF** at (28.7, 53.3)
- removed the REF** at (268.5, 153.3)
- removed the REF** at (205.3, 53.3)
- removed the REF** at (91.9, 153.3)
- removed the U1 at (69.4, 129.5)
- removed the U1 at (246.0, 129.5)
- removed the U3 at (246.5, 87.3)
- removed the U3 at (70.0, 87.3)
- removed the U4 at (69.4, 96.5)
- removed the U4 at (246.0, 96.5)
- removed the U6 at (268.6, 98.5)
- removed the U6 at (92.1, 98.5)
- added G***: LOGO, Symbol:Logo_Preto - Copia, F.Cu at (256.8, 71.3)
- added G***: LOGO, Symbol:Logo_Preto - Copia, F.Cu at (96.8, 70.8)
- added J1: Power Supply, TerminalBlock:TerminalBlock_bornier-2_P5.08mm, F.Cu at (54.3, 55.5)
- added J1: Power Supply, TerminalBlock:TerminalBlock_bornier-2_P5.08mm, F.Cu at (82.3, 152.0)
- added J1: Power Supply, TerminalBlock:TerminalBlock_bornier-2_P5.08mm, F.Cu at (214.3, 56.0)
- added J1: Power Supply, TerminalBlock:TerminalBlock_bornier-2_P5.08mm, F.Cu at (242.3, 152.5)
- added J2: Conn_01x03_Male, TerminalBlock:TerminalBlock_bornier-3_P5.08mm, F.Cu at (70.8, 152.0)
- added J2: Conn_01x03_Male, TerminalBlock:TerminalBlock_bornier-3_P5.08mm, F.Cu at (230.8, 152.5)
- added J3: Conn_01x03_Male, TerminalBlock:TerminalBlock_bornier-3_P5.08mm, F.Cu at (64.5, 55.5)
- added J3: Conn_01x03_Male, TerminalBlock:TerminalBlock_bornier-3_P5.08mm, F.Cu at (224.5, 56.0)
- added REF**: MountingHole_2.2mm_M2, MountingHole:MountingHole_2.2mm_M2, F.Cu at (101.2, 52.9)
- added REF**: MountingHole_2.2mm_M2, MountingHole:MountingHole_2.2mm_M2, F.Cu at (198.0, 53.3)
- added REF**: MountingHole_2.2mm_M2, MountingHole:MountingHole_2.2mm_M2, F.Cu at (38.0, 152.9)
- added REF**: MountingHole_2.2mm_M2, MountingHole:MountingHole_2.2mm_M2, F.Cu at (261.2, 153.3)
- added REF**: MountingHole_2.2mm_M2, MountingHole:MountingHole_2.2mm_M2, F.Cu at (198.0, 153.3)
- added REF**: MountingHole_2.2mm_M2, MountingHole:MountingHole_2.2mm_M2, F.Cu at (101.2, 152.9)
- added REF**: MountingHole_2.2mm_M2, MountingHole:MountingHole_2.2mm_M2, F.Cu at (38.0, 52.9)
- added REF**: MountingHole_2.2mm_M2, MountingHole:MountingHole_2.2mm_M2, F.Cu at (261.2, 53.3)
- added U1: ESP32-DEVKIT-V1, ESP32-DEVKIT-V1:MODULE_ESP32_DEVKIT_V1, F.Cu at (78.7, 129.1)
- added U1: ESP32-DEVKIT-V1, ESP32-DEVKIT-V1:MODULE_ESP32_DEVKIT_V1, F.Cu at (238.7, 129.6)
- added U3: FlashMemory_W25Q128, Jupiter:FlashMemory W25Q128, F.Cu at (79.2, 86.9)
- added U3: FlashMemory_W25Q128, Jupiter:FlashMemory W25Q128, F.Cu at (239.2, 87.4)
- added U4: GY-521 - Sensor 1, GY-521:GY-521, F.Cu at (238.7, 96.6)
- added U4: GY-521 - Sensor 1, GY-521:GY-521, F.Cu at (78.7, 96.1)
- added U6: GY-BMP280, Jupiter:GY BMP280, F.Cu at (88.3, 95.2)
- added U6: GY-BMP280, Jupiter:GY BMP280, F.Cu at (248.3, 95.6)
- moved G*** 58.5 mm to (177.1, 71.2), turned to -90 degrees
- moved U6 13.4 mm to (168.6, 95.5), turned to 0 degrees
Routing:
- net /PWM 2: track 557.5 -> 356.3 mm
- net /SDA: track 323.6 -> 122.6 mm, vias 6 -> 0
- net /3v3: track 257.6 -> 162.6 mm, vias 9 -> 0
- net /HMOSI: track 399.1 -> 341.3 mm, vias 6 -> 0
- net /CS: track 359.2 -> 407.7 mm
- net /HMISO: track 453.5 -> 406.9 mm, vias 9 -> 6
- net /SCL: track 183.6 -> 225.1 mm
- net /HCLK: track 341.1 -> 371.0 mm
- net VCC: track 518.2 -> 510.8 mm
- net GND: track 2.30 -> 0.00 mm
- added copper zone on B.Cu, net GND
Other:
- board size 249.7 x 110 mm -> 73.2 x 110 mm
