File: Projeto Elétrico - ControleTrix.kicad_pcb (KiCad board)
At the start: 2 copper layers, 55.1 x 87.3 mm, 15 parts, among them J1 Power Supply, J2 Conn_01x03_Male, J3 Conn_01x03_Male, U1 ESP32-DEVKIT-V1, U3 FlashMemory, U4 GY-521 - Sensor 1, U6 GY-BMP280

Commit message: Add files via upload
Atualização da posição dos bornes
Parts:
- moved J2 78.2 mm to (118.1, 72.4), turned to 0 degrees
- moved J3 15.7 mm to (146.1, 72.4)
- moved J1 15.3 mm to (139.7, 74.9)
- moved J1 9.90 mm to (134.6, 147.3)
Routing:
- net /PWM 1: track 8.95 -> 98.9 mm
- net VCC: track 124.9 -> 53.5 mm
- net /PWM 2: track 48.4 -> 65.9 mm
Changed lines of the file:
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@@
   (net 32 "unconnected-(U1-Pad25)")
   (footprint "TerminalBlock:TerminalBlock_bornier-2_P5.08mm" (layer "F.Cu")
-    (at 124.46 76.2 180)
+    (at 139.7 74.93 180)
     (descr "simple 2-pin terminal block, pitch 5.08mm, revamped version of bornier2")
     (tags "terminal block bornier2")
@@
   )
   (footprint "TerminalBlock:TerminalBlock_bornier-3_P5.08mm" (layer "F.Cu")
-    (at 135.55 148.59 180)
+    (at 118.11 72.39)
     (descr "simple 3-pin terminal block, pitch 5.08mm, revamped version of bornier3")
     (tags "terminal block bornier3")
@@
     (fp_line (start 12.63 3.75) (end -2.47 3.75)
       (stroke (width 0.1) (type solid)) (layer "F.Fab"))
-    (pad "1" thru_hole rect (at 0 0 180) (size 3 3) (drill 1.52) (layers "*.Cu" "*.Mask")
+    (pad "1" thru_hole rect (at 0 0) (size 3 3) (drill 1.52) (layers "*.Cu" "*.Mask")
       (net 3 "/PWM 1") (pinfunction "Pin_1") (pintype "passive"))
-    (pad "2" thru_hole circle (at 5.08 0 180) (size 3 3) (drill 1.52) (layers "*.Cu" "*.Mask")
+    (pad "2" thru_hole circle (at 5.08 0) (size 3 3) (drill 1.52) (layers "*.Cu" "*.Mask")
       (net 2 "VCC") (pinfunction "Pin_2") (pintype "passive"))
-    (pad "3" thru_hole circle (at 10.16 0 180) (size 3 3) (drill 1.52) (layers "*.Cu" "*.Mask")
+    (pad "3" thru_hole circle (at 10.16 0) (size 3 3) (drill 1.52) (layers "*.Cu" "*.Mask")
       (net 1 "GND") (pinfunction "Pin_3") (pintype "passive"))
     (model "${KICAD6_3DMODEL_DIR}/TerminalBlock.3dshapes/TerminalBlock_bornier-3_P5.08mm.wrl"
@@
   )
   (footprint "TerminalBlock:TerminalBlock_bornier-2_P5.08mm" (layer "F.Cu")
-    (at 144.44 148.59)
+    (at 134.62 147.32)
     (descr "simple 2-pin terminal block, pitch 5.08mm, revamped version of bornier2")
     (tags "terminal block bornier2")
@@
   )
   (footprint "TerminalBlock:TerminalBlock_bornier-3_P5.08mm" (layer "F.Cu")
-    (at 130.81 76.2)
+    (at 146.05 72.39)
     (descr "simple 3-pin terminal block, pitch 5.08mm, revamped version of bornier3")
     (tags "terminal block bornier3")
@@
     (style (thickness 0.1) (arrow_length 1.27) (text_position_mode 2) (extension_height 0.58642) (extension_offset 0.5) keep_text_aligned)
   )
-  (segment (start 134.62 72.39) (end 135.89 73.66) (width 1) (layer "B.Cu") (net 2))
-  (segment (start 119.38 76.2) (end 119.38 78.74) (width 1) (layer "B.Cu") (net 2))
-  (segment (start 119.38 76.2) (end 119.38 73.66) (width 1) (layer "B.Cu") (net 2))
-  (segment (start 119.38 78.74) (end 118.11 80.01) (width 1) (layer "B.Cu") (net 2))
-  (segment (start 120.65 72.39) (end 134.62 72.39) (width 1) (layer "B.Cu") (net 2))
-  (segment (start 113.96 144.78) (end 126.66 144.78) (width 1) (layer "B.Cu") (net 2))
-  (segment (start 126.66 144.78) (end 130.47 148.59) (width 1) (layer "B.Cu") (net 2))
+  (segment (start 150.79 147.32) (end 153.605 144.505) (width 1) (layer "B.Cu") (net 2))
+  (segment (start 134.62 71.12) (end 135.89 69.85) (width 1) (layer "B.Cu") (net 2))
+  (segment (start 134.62 74.93) (end 134.62 71.12) (width 1) (layer "B.Cu") (net 2))
+  (segment (start 148.59 69.85) (end 151.13 72.39) (width 1) (layer "B.Cu") (net 2))
   (segment (start 153.605 144.505) (end 153.605 140.97) (width 1) (layer "B.Cu") (net 2))
-  (segment (start 114.3 80.01) (end 111.76 82.55) (width 1) (layer "B.Cu") (net 2))
-  (segment (start 149.52 148.59) (end 153.605 144.505) (width 1) (layer "B.Cu") (net 2))
-  (segment (start 111.76 82.55) (end 111.76 142.58) (width 1) (layer "B.Cu") (net 2))
-  (segment (start 119.38 73.66) (end 120.65 72.39) (width 1) (layer "B.Cu") (net 2))
-  (segment (start 118.11 80.01) (end 114.3 80.01) (width 1) (layer "B.Cu") (net 2))
-  (segment (start 135.89 73.66) (end 135.89 76.2) (width 1) (layer "B.Cu") (net 2))
-  (segment (start 111.76 142.58) (end 113.96 144.78) (width 1) (layer "B.Cu") (net 2))
-  (segment (start 133.285 140.97) (end 133.285 146.325) (width 1) (layer "B.Cu") (net 3))
-  (segment (start 133.285 146.325) (end 135.55 148.59) (width 1) (layer "B.Cu") (net 3))
-  (segment (start 133.01 141.245) (end 133.285 140.97) (width 0.25) (layer "B.Cu") (net 3))
-  (segment (start 133.093 112.903) (end 133.285 113.095) (width 1) (layer "F.Cu") (net 4))
-  (segment (start 125.2555 84.3) (end 125.349 84.3935) (width 1) (layer "F.Cu") (net 4))
+  (segment (start 133.35 69.85) (end 125.73 69.85) (width 1) (layer "B.Cu") (net 2))
+  (segment (start 134.62 71.12) (end 133.35 69.85) (width 1) (layer "B.Cu") (net 2))
+  (segment (start 139.7 147.32) (end 150.79 147.32) (width 1) (layer "B.Cu") (net 2))
+  (segment (start 135.89 69.85) (end 148.59 69.85) (width 1) (layer "B.Cu") (net 2))
+  (segment (start 123.19 72.39) (end 125.73 69.85) (width 1) (layer "B.Cu") (net 2))
+  (segment (start 113.03 144.78) (end 111.76 143.51) (width 1) (layer "B.Cu") (net 3))
+  (segment (start 118.11 72.39) (end 118.11 74.93) (width 1) (layer "B.Cu") (net 3))
+  (segment (start 132.08 144.78) (end 113.03 144.78) (width 1) (layer "B.Cu") (net 3))
+  (segment (start 111.76 143.51) (end 111.76 81.28) (width 1) (layer "B.Cu") (net 3))
+  (segment (start 133.285 140.97) (end 133.285 143.575) (width 1) (layer "B.Cu") (net 3))
+  (segment (start 133.285 143.575) (end 132.08 144.78) (width 1) (layer "B.Cu") (net 3))
+  (segment (start 118.11 74.93) (end 111.76 81.28) (width 1) (layer "B.Cu") (net 3))
   (segment (start 127.254 112.903) (end 133.093 112.903) (width 1) (layer "F.Cu") (net 4))
+  (segment (start 125.349 87.63) (end 125.349 110.998) (width 1) (layer "F.Cu") (net 4))
+  (segment (start 133.093 112.903) (end 133.285 113.095) (width 1) (layer "F.Cu") (net 4))
   (segment (start 125.349 110.998) (end 127.254 112.903) (width 1) (layer "F.Cu") (net 4))
-  (segment (start 125.349 84.3935) (end 125.349 110.998) (width 1) (layer "F.Cu") (net 4))
-  (via (at 125.2555 84.3) (size 1.5) (drill 0.8) (layers "F.Cu" "B.Cu") (net 4))
+  (via (at 125.349 87.63) (size 1.5) (drill 0.8) (layers "F.Cu" "B.Cu") (net 4))
   (via (at 133.285 113.095) (size 1.5) (drill 0.8) (layers "F.Cu" "B.Cu") (net 4))
-  (segment (start 125.2555 84.3) (end 125.73 83.8255) (width 1) (layer "B.Cu") (net 4))
-  (segment (start 125.73 83.82) (end 130.81 78.74) (width 1) (layer "B.Cu") (net 4))
-  (segment (start 130.81 78.74) (end 130.81 76.2) (width 1) (layer "B.Cu") (net 4))
-  (segment (start 125.73 83.8255) (end 125.73 83.82) (width 1) (layer "B.Cu") (net 4))
+  (segment (start 127 83.82) (end 125.349 85.471) (width 1) (layer "B.Cu") (net 4))
+  (segment (start 125.349 85.471) (end 125.349 87.63) (width 1) (layer "B.Cu") (net 4))
+  (segment (start 146.05 77.47) (end 139.7 83.82) (width 1) (layer "B.Cu") (net 4))
+  (segment (start 146.05 72.39) (end 146.05 77.47) (width 1) (layer "B.Cu") (net 4))
   (segment (start 133.285 115.57) (end 133.285 113.095) (width 1) (layer "B.Cu") (net 4))
+  (segment (start 139.7 83.82) (end 127 83.82) (width 1) (layer "B.Cu") (net 4))
   (segment (start 152.366 97.756) (end 150.685 97.756) (width 1) (layer "B.Cu") (net 5))
   (segment (start 153.605 115.57) (end 153.605 98.995) (width 1) (layer "B.Cu") (net 5))
